File: Breakout Boards/ICs-1.brd (EAGLE design)
At the start: 150 x 75 mm, 51 parts

Commit message: new
Other:
- board size 150 x 75 mm -> 170 x 95 mm
- board text added: "Breakout Boards"
- board text added: "SOLDER MASK"
- board text added: "TOP SOLDER"
