File: Tube Prototypes/counter-test.sch (EAGLE design)
At the start: 16 parts

Commit message: new
Parts:
- removed RESET-10S, U$4: SWITCH-MOMENTARY4MM, iStivi - Button-Switch:SWITCH-MOMENTARY4MM
Connections:
- new net VCC: RESET-1S.1, U$3.1, U$5.1
- net N$14: now also U$5.2
- net N$19: now also RESET-1S.2
- net N$7: now also U$3.2
Changed lines of the file:
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@@
 <part name="GND4" library="iStivi - Supply" deviceset="GND" device=""/>
 <part name="RESET-1S" library="iStivi - Button-Switch" deviceset="SWITCH-MOMENTARY" device="4MM"/>
-<part name="RESET-10S" library="iStivi - Button-Switch" deviceset="SWITCH-MOMENTARY" device="4MM"/>
 <part name="U$3" library="iStivi - Button-Switch" deviceset="SWITCH-MOMENTARY" device="4MM"/>
-<part name="U$4" library="iStivi - Button-Switch" deviceset="SWITCH-MOMENTARY" device="4MM"/>
 <part name="U$5" library="iStivi - Button-Switch" deviceset="SWITCH-MOMENTARY" device="4MM"/>
+<part name="P+1" library="iStivi - Supply" deviceset="VCC" device=""/>
 </parts>
 <sheets>
@@
 <instance part="GND4" gate="1" x="-17.78" y="38.1"/>
 <instance part="RESET-1S" gate="G$1" x="149.86" y="17.78" rot="R90"/>
-<instance part="RESET-10S" gate="G$1" x="114.3" y="17.78" rot="R90"/>
 <instance part="U$3" gate="G$1" x="60.96" y="17.78" rot="R90"/>
-<instance part="U$4" gate="G$1" x="27.94" y="17.78" rot="R90"/>
 <instance part="U$5" gate="G$1" x="-25.4" y="17.78" rot="R90"/>
+<instance part="P+1" gate="VCC" x="43.18" y="5.08" rot="R180"/>
 </instances>
 <busses>
@@
 <pinref part="1H" gate="G$1" pin="4"/>
 <pinref part="IC-1H" gate="A" pin="QD"/>
-<wire x1="-27.94" y1="88.9" x2="-27.94" y2="73.66" width="0.1524" layer="91"/>
+<wire x1="-27.94" y1="88.9" x2="-27.94" y2="81.28" width="0.1524" layer="91"/>
+<wire x1="-27.94" y1="81.28" x2="-27.94" y2="73.66" width="0.1524" layer="91"/>
+<wire x1="-27.94" y1="81.28" x2="-53.34" y2="81.28" width="0.1524" layer="91"/>
+<wire x1="-53.34" y1="81.28" x2="-53.34" y2="33.02" width="0.1524" layer="91"/>
+<junction x="-27.94" y="81.28"/>
+<wire x1="-53.34" y1="33.02" x2="-71.12" y2="33.02" width="0.1524" layer="91"/>
+<wire x1="-71.12" y1="33.02" x2="-71.12" y2="48.26" width="0.1524" layer="91"/>
 </segment>
 </net>
@@
 <junction x="111.76" y="81.28"/>
 <pinref part="IC-1M" gate="A" pin="CKA"/>
-<wire x1="76.2" y1="33.02" x2="50.8" y2="33.02" width="0.1524" layer="91"/>
+<wire x1="76.2" y1="33.02" x2="60.96" y2="33.02" width="0.1524" layer="91"/>
+<wire x1="60.96" y1="33.02" x2="50.8" y2="33.02" width="0.1524" layer="91"/>
 <wire x1="50.8" y1="33.02" x2="50.8" y2="48.26" width="0.1524" layer="91"/>
+<pinref part="U$3" gate="G$1" pin="2"/>
+<wire x1="60.96" y1="22.86" x2="60.96" y2="33.02" width="0.1524" layer="91"/>
+<junction x="60.96" y="33.02"/>
 </segment>
 </net>
@@
 <junction x="25.4" y="81.28"/>
 <pinref part="IC-1H" gate="A" pin="CKA"/>
-<wire x1="-10.16" y1="33.02" x2="-35.56" y2="33.02" width="0.1524" layer="91"/>
+<wire x1="-10.16" y1="33.02" x2="-25.4" y2="33.02" width="0.1524" layer="91"/>
+<wire x1="-25.4" y1="33.02" x2="-35.56" y2="33.02" width="0.1524" layer="91"/>
 <wire x1="-35.56" y1="33.02" x2="-35.56" y2="48.26" width="0.1524" layer="91"/>
+<pinref part="U$5" gate="G$1" pin="2"/>
+<wire x1="-25.4" y1="22.86" x2="-25.4" y2="33.02" width="0.1524" layer="91"/>
+<junction x="-25.4" y="33.02"/>
 </segment>
 </net>
@@
 <pinref part="IC-1S" gate="A" pin="CKA"/>
 <pinref part="JP1" gate="G$1" pin="1"/>
-<wire x1="139.7" y1="48.26" x2="139.7" y2="-7.62" width="0.1524" layer="91"/>
+<wire x1="139.7" y1="48.26" x2="139.7" y2="33.02" width="0.1524" layer="91"/>
+<wire x1="139.7" y1="33.02" x2="139.7" y2="-7.62" width="0.1524" layer="91"/>
 <wire x1="139.7" y1="-7.62" x2="147.32" y2="-7.62" width="0.1524" layer="91"/>
+<pinref part="RESET-1S" gate="G$1" pin="2"/>
+<wire x1="149.86" y1="22.86" x2="149.86" y2="33.02" width="0.1524" layer="91"/>
+<wire x1="149.86" y1="33.02" x2="139.7" y2="33.02" width="0.1524" layer="91"/>
+<junction x="139.7" y="33.02"/>
 </segment>
 </net>
@@
 </segment>
 </net>
+<net name="VCC" class="0">
+<segment>
+<pinref part="U$5" gate="G$1" pin="1"/>
+<pinref part="U$3" gate="G$1" pin="1"/>
+<wire x1="-25.4" y1="12.7" x2="43.18" y2="12.7" width="0.1524" layer="91"/>
+<pinref part="RESET-1S" gate="G$1" pin="1"/>
+<wire x1="43.18" y1="12.7" x2="60.96" y2="12.7" width="0.1524" layer="91"/>
+<wire x1="60.96" y1="12.7" x2="149.86" y2="12.7" width="0.1524" layer="91"/>
+<junction x="60.96" y="12.7"/>
+<pinref part="P+1" gate="VCC" pin="VCC"/>
+<wire x1="43.18" y1="7.62" x2="43.18" y2="12.7" width="0.1524" layer="91"/>
+<junction x="43.18" y="12.7"/>
+</segment>
+</net>
