File: Tube Prototypes/tube-tester.brd (EAGLE design)
At the start: 100 x 75 mm, 37 parts, among them IC1 NE555D, IC2 74141N, IC3 7805TV, Q1 IRF740S, Q2 BC546B

Commit message: new
Parts:
- IC3: value 7805TV -> 7805
- Q2: value BC546B -> BC546
- R6: value (none) -> 2K2

Commit message: tube tester
Other:
- board size 100 x 75 mm -> 120 x 95 mm
- board text added: "BOTTOM MASK"
- board text added: "BOTTOM SOLDER"
- board text added: "SILK SCREEN"
- board text added: "TOP MASK"
- board text added: "TOP SOLDER"
Changed lines of the file:
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@@
 <setting verticaltext="up"/>
 </settings>
-<grid distance="0.5" unitdist="mm" unit="mm" style="lines" multiple="1" display="no" altdistance="0.025" altunitdist="inch" altunit="inch"/>
+<grid distance="5" unitdist="mm" unit="mm" style="lines" multiple="1" display="no" altdistance="0.025" altunitdist="inch" altunit="inch"/>
 <layers>
-<layer number="1" name="Top" color="4" fill="1" visible="no" active="yes"/>
+<layer number="1" name="Top" color="4" fill="1" visible="yes" active="yes"/>
 <layer number="2" name="Route2" color="1" fill="3" visible="no" active="no"/>
 <layer number="3" name="Route3" color="4" fill="3" visible="no" active="no"/>
 <layer number="14" name="Route14" color="1" fill="6" visible="no" active="no"/>
 <layer number="15" name="Route15" color="4" fill="6" visible="no" active="no"/>
-<layer number="16" name="Bottom" color="1" fill="1" visible="no" active="yes"/>
+<layer number="16" name="Bottom" color="1" fill="1" visible="yes" active="yes"/>
 <layer number="17" name="Pads" color="2" fill="1" visible="yes" active="yes"/>
 <layer number="18" name="Vias" color="2" fill="1" visible="yes" active="yes"/>
@@
 <layer number="27" name="tValues" color="7" fill="1" visible="yes" active="yes"/>
 <layer number="28" name="bValues" color="7" fill="1" visible="yes" active="yes"/>
-<layer number="29" name="tStop" color="7" fill="3" visible="yes" active="yes"/>
-<layer number="30" name="bStop" color="7" fill="6" visible="yes" active="yes"/>
+<layer number="29" name="tStop" color="7" fill="1" visible="yes" active="yes"/>
+<layer number="30" name="bStop" color="7" fill="1" visible="yes" active="yes"/>
 <layer number="31" name="tCream" color="7" fill="4" visible="yes" active="yes"/>
 <layer number="32" name="bCream" color="7" fill="5" visible="yes" active="yes"/>
@@
 <text x="96.52" y="62.23" size="1.778" layer="16" rot="SMR270">TUBE TESTER</text>
 <text x="96.52" y="44.45" size="1.778" layer="1" rot="SR90">TUBE TESTER</text>
+<wire x1="0" y1="0" x2="-10" y2="0" width="0.4064" layer="20"/>
+<wire x1="-10" y1="0" x2="0" y2="-10" width="0.4064" layer="20"/>
+<wire x1="0" y1="-10" x2="0" y2="0" width="0.4064" layer="20"/>
+<wire x1="100" y1="0" x2="100" y2="-10" width="0.4064" layer="20"/>
+<wire x1="100" y1="-10" x2="110" y2="0" width="0.4064" layer="20"/>
+<wire x1="110" y1="0" x2="100" y2="0" width="0.4064" layer="20"/>
+<wire x1="100" y1="75" x2="100" y2="85" width="0.4064" layer="20"/>
+<wire x1="100" y1="85" x2="110" y2="75" width="0.4064" layer="20"/>
+<wire x1="110" y1="75" x2="100" y2="75" width="0.4064" layer="20"/>
+<wire x1="0" y1="75" x2="0" y2="85" width="0.4064" layer="20"/>
+<wire x1="0" y1="85" x2="-10" y2="75" width="0.4064" layer="20"/>
+<wire x1="-10" y1="75" x2="0" y2="75" width="0.4064" layer="20"/>
+<text x="15" y="80" size="1.778" layer="20">TUBE TESTER</text>
+<text x="55" y="80" size="1.778" layer="1">TOP SOLDER</text>
+<text x="75" y="80" size="1.778" layer="16" rot="MR0">BOTTOM SOLDER</text>
+<text x="55" y="80" size="1.778" layer="29">TOP MASK</text>
+<text x="75" y="80" size="1.778" layer="30" rot="MR0">BOTTOM MASK</text>
+<text x="55" y="80" size="1.778" layer="25">SILK SCREEN</text>
 </plain>
 <attributes>
