File: Tube Prototypes/tube-tester.sch (EAGLE design)
At the start: 33 parts, among them IC1 NE555D, IC2 74141N, IC3 7805TV, Q1 IRF740S, Q2 BC546B

Commit message: new
Parts:
- IC3: value 7805TV -> 7805
- Q2: value BC546B -> BC546
- R6: value (none) -> 2K2
Changed lines of the file:
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@@
 <part name="R5" library="iStivi - RCLD" deviceset="RESISTOR" device="0207/10" value="220K"/>
 <part name="R4" library="iStivi - RCLD" deviceset="RESISTOR" device="0207/10" value="470R"/>
-<part name="R6" library="iStivi - RCLD" deviceset="RESISTOR" device="R1206"/>
+<part name="R6" library="iStivi - RCLD" deviceset="RESISTOR" device="R1206" value="2K2"/>
 <part name="C3" library="iStivi - RCLD" deviceset="CAPACITOR" device="C1206K" value="100pF"/>
-<part name="Q2" library="iStivi - Transistor-FET" deviceset="BC546*" device="" technology="B"/>
+<part name="Q2" library="iStivi - Transistor-FET" deviceset="BC546*" device="" technology="B" value="BC546"/>
 <part name="C2" library="iStivi - RCLD" deviceset="CAPACITOR" device="C1206K" value="2n2"/>
 <part name="L1" library="iStivi - RCLD" deviceset="INDUCTOR" device="0207/10" value="100uH"/>
@@
 <part name="C" library="iStivi - Button-Switch" deviceset="320-916" device=""/>
 <part name="D" library="iStivi - Button-Switch" deviceset="320-916" device=""/>
-<part name="IC3" library="iStivi - Transistor-FET-reg" deviceset="78*" device="TV" technology="05"/>
+<part name="IC3" library="iStivi - Transistor-FET-reg" deviceset="78*" device="TV" technology="05" value="7805"/>
 <part name="JP1" library="iStivi - Header-Connector" deviceset="M02" device="3.5MM"/>
 <part name="C5" library="iStivi - RCLD" deviceset="CAPACITOR_POL" device="E2-5" value="100uF"/>

Commit message: new ignore
Connections:
- net GND: now also Q1.S
Changed lines of the file:
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@@
 <wire x1="91.44" y1="15.24" x2="81.28" y2="15.24" width="0.1524" layer="91"/>
 <wire x1="81.28" y1="15.24" x2="66.04" y2="15.24" width="0.1524" layer="91"/>
-<wire x1="66.04" y1="15.24" x2="38.1" y2="15.24" width="0.1524" layer="91"/>
+<wire x1="66.04" y1="15.24" x2="48.26" y2="15.24" width="0.1524" layer="91"/>
+<wire x1="48.26" y1="15.24" x2="38.1" y2="15.24" width="0.1524" layer="91"/>
 <wire x1="81.28" y1="48.26" x2="81.28" y2="15.24" width="0.1524" layer="91"/>
 <junction x="81.28" y="15.24"/>
@@
 <wire x1="236.22" y1="25.4" x2="236.22" y2="15.24" width="0.1524" layer="91"/>
 <junction x="236.22" y="15.24"/>
+<pinref part="Q1" gate="G$1" pin="S"/>
+<wire x1="48.26" y1="55.88" x2="48.26" y2="15.24" width="0.1524" layer="91"/>
+<junction x="48.26" y="15.24"/>
 </segment>
 </net>
