File: Tube Prototypes/tube-tester.job.brd (EAGLE design)
At the start: 100 x 100 mm, 36 parts, among them IC1 NE555D, IC2 74141N, IC3 7805, Q1 IRF740S, Q2 BC546

Commit message: tube tester redo
Routing:
- net N$22: track 176.1 -> 75.1 mm, vias 2 -> 0
- net N$23: track 140.5 -> 57.1 mm, vias 3 -> 2
- net N$13: track 101.1 -> 130.0 mm, vias 1 -> 0
- net N$24: track 44.2 -> 66.6 mm, vias 3 -> 1
- net N$5: track 45.7 -> 67.3 mm, vias 0 -> 2
- net N$26: track 152.1 -> 132.8 mm
- net N$3: track 37.3 -> 52.7 mm, vias 2 -> 0
- net N$16: track 101.3 -> 86.0 mm, vias 1 -> 0
- net N$14: track 93.9 -> 109.2 mm, vias 3 -> 1
- net N$1: track 24.2 -> 39.2 mm, vias 2 -> 0
- net N$4: track 38.8 -> 25.9 mm, vias 2 -> 0
- net N$30: track 82.6 -> 95.0 mm, vias 3 -> 5
- net N$18: track 55.2 -> 43.9 mm, vias 0 -> 1
- net N$29: track 100.3 -> 109.8 mm, vias 0 -> 1
- net GND: track 298.1 -> 304.4 mm, vias 3 -> 1
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Other:
- board text added: "DESGINED & PRODUCED S. MARTIN"
- board text added: "NIXIE TESTER BOARD"
- board text removed: "DESIGNED & PRODUCED S. MARTIN"
- board text removed: "NIXIE TUBE TEST BOARD"
