File: clock tests/clock_prototype.sch (EAGLE design)
At the start: 37 parts, among them IC1 74LS14N, IC2 74LS08N, IC3 74LS08N, IC4 74LS11N, IC5 74LS32N, IC6 74LS112D

Commit message: clock update
Parts:
- removed 10HOURS: 74LS92N, iStivi - ICs:74LS92N
- removed AM/PM: (no value), iStivi - Button-Switch:320-916
- removed RESET: SWITCH-MOMENTARY12MM, iStivi - Button-Switch:SWITCH-MOMENTARY12MM
- added IC7: 74S260N, iStivi - ICs:74S260N
- added IC8: 74LS32N, iStivi - ICs:74LS32N
- C1, C2: value 15pF -> 22pF
- Q1: value (none) -> 32.768Hz
- R1: value 1M -> 10M
- R2: value 1K -> 330K
Connections:
- removed net 10H_A: 10H.1, 10HOURSA.QA, IC3A.I0
- new net N$10: IC4A.O, IC5D.I1
- new net N$22: IC7A.O, IC8A.I1
- new net N$24: IC2B.O, IC8A.I0
- new net N$8: IC1F.O, IC6B.!CLR
- new net N$9: IC5C.I0, IC5D.O
- net 10H_B: now also IC3B.I0, IC6B.!Q; no longer 10HOURSA.QB, IC4A.I0
- net 1H_A: now also IC4A.I1, IC7A.I1
- net 1H_B: now also IC7A.I2; no longer IC3A.I1
- net 1H_C: now also IC3B.I1, IC7A.I3
- net 1H_D: now also IC6B.CLK, IC7A.I4; no longer 10HOURSA.CKA, IC4A.I1
- net GND: no longer R3.2
- net N$14: now also U$1G$1.RCLK
- net N$16: now also R3.1, U$1G$1.Q6; no longer U$1G$1.Q7
- net N$25: now also IC1F.I; no longer 10HOURSA.R0(1), 10HOURSA.R0(2)
- net N$27: no longer AM/PM.O, IC3A.O
- net N$28: now also IC3B.O, IC5D.I0; no longer AM/PM.S, IC4A.O
- net N$3: now also IC8A.O; no longer IC2B.O
- net N$5: now also 10H.1, IC4A.I0, IC6B.Q, IC7A.I0; no longer AM/PM.P, IC5C.I0
- net N$6: no longer RESET.2
- net VCC: now also R3.2; no longer R3.1, RESET.1
Other:
- note removed: "12/24 HOUR TYPE"
- moved on the sheet: IC4A, R3
