File: clock tests/clock_pulse_test.sch (EAGLE design)
At the start: 12 parts, among them IC1 74LS14N, Q1 32.768kHz

Commit message: clock pulse test new
Parts:
- IC1: value 74LS14N -> 74LS14D; device iStivi - ICs:74LS14N -> iStivi - ICs:74LS14D
Changed lines of the file:
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@@
 <parts>
 <part name="Q1" library="iStivi - Oscillators" deviceset="CRYSTAL" device="TC26V" value="32.768kHz"/>
-<part name="IC1" library="iStivi - ICs" deviceset="74*14" device="N" technology="LS"/>
+<part name="IC1" library="iStivi - ICs" deviceset="74*14" device="D" technology="LS" value="74LS14D"/>
 <part name="C2" library="iStivi - RCLD" deviceset="CAPACITOR" device="050-024X044" value="22pF"/>
 <part name="R1" library="iStivi - RCLD" deviceset="RESISTOR" device="0207/10" value="10M"/>
