File: clock tests/counter_test.sch (EAGLE design)
At the start: 36 parts, among them IC1 74LS14N, IC2 74LS08N, IC3 74LS08N, IC4 74LS11N, IC5 74LS32N, IC6 74LS112D, IC7 74S260N, IC8 74LS32N, Q1 32.768Hz

Commit message: new
Parts:
- removed C2: 22pF, iStivi - RCLD:CAPACITOR050-024X044
- removed IC1: 74LS14N, iStivi - ICs:74LS14N
- removed IC2: 74LS08N, iStivi - ICs:74LS08N
- removed IC7: 74S260N, iStivi - ICs:74S260N
- removed IC8: 74LS32N, iStivi - ICs:74LS32N
- removed JP1: (no value), iStivi - Header-Connector:M02PTH
- removed Q1: 32.768Hz, iStivi - Oscillators:CRYSTALTC26V
- removed R1: 10M, iStivi - RCLD:RESISTOR0207/7
- removed R2: 330K, iStivi - RCLD:RESISTOR0207/7
- removed R3, R4: 10K, iStivi - RCLD:RESISTOR0207/7
- removed R5, R6, R7, R8: 4K7, iStivi - RCLD:RESISTOR0207/7
- removed SET, SET_HR, SET_MIN: SWITCH-MOMENTARY12MM, iStivi - Button-Switch:SWITCH-MOMENTARY12MM
- removed U$1: 748154D, iStivi - ICs:748154D
- added 10HOURS: 74LS92N, iStivi - ICs:74LS92N
- added AM_PM, HOUR_COUNT, MIN_COUNT, POWER: (no value), iStivi - Header-Connector:M02PTH3
- added CLOCK_IN, HR_RESET: M01PTH_LONGPAD, iStivi - Header-Connector:M01PTH_LONGPAD
- added HOUR_SET: (no value), iStivi - Header-Connector:M03LONGPADS
- 10H: device iStivi - Header-Connector:M02PTH -> iStivi - Header-Connector:M02PTH3
- 10M, 10S: device iStivi - Header-Connector:M03PTH -> iStivi - Header-Connector:M03LONGPADS
- 1H, 1M, 1S: device iStivi - Header-Connector:M04PTH -> iStivi - Header-Connector:M04LONGPADS
- C1: value 22pF -> 330uF; device iStivi - RCLD:CAPACITOR050-024X044 -> iStivi - RCLD:CAPACITOR_POLE3.5-8
- IC5: value 74LS32N -> 74S260D; device iStivi - ICs:74LS32N -> iStivi - ICs:74S260D
Connections:
- removed net N$10: IC4A.O, IC5D.I1
- removed net N$11: C1.1, IC1A.I, Q1.1, R1.2
- removed net N$12: C2.1, Q1.2, R2.2
- removed net N$13: IC1A.O, IC1B.I, R1.1, R2.1
- removed net N$14: IC1B.O, R4.1, U$1G$1.CLKA, U$1G$1.RCLK
- removed net N$16: IC2D.I1, R3.1, U$1G$1.Q6
- removed net N$17: IC1D.O, IC2D.I0
- removed net N$18: IC1C.I, IC1D.I, IC2A.I1, IC2C.I0, R5.2, R6.2, SET.2
- removed net N$19: IC2C.I1, SET_MIN.2
- removed net N$20: IC1C.O, IC2B.I0
- removed net N$22: IC7A.O, IC8A.I1
- removed net N$23: IC2A.I0, R7.2, SET_HR.2
- removed net N$24: IC2B.O, IC8A.I0
- removed net N$25: HOURSA.R0(1), HOURSA.R0(2), IC1F.I, IC5C.O
- removed net N$27: IC6A.CLK
- removed net N$28: IC3B.O, IC5D.I0
- removed net N$3: IC5B.I1, IC8A.O
- removed net N$4: IC2A.O, IC5B.I0
- removed net N$5: 10H.1, IC4A.I0, IC6B.Q, IC7A.I0
- removed net N$6: 10MINUTESA.R0(1), 10MINUTESA.R0(2), 10SECONDSA.R0(1), 10SECONDSA.R0(2), IC5C.I1, MINUTESA.R0(1), MINUTESA.R0(2), R8.2, SECONDSA.R0(1), SECONDSA.R0(2)
- removed net N$7: IC6A.!CLR, IC6A.!PRE, IC6A.J, IC6A.K, R9.2
- removed net N$8: IC1F.O, IC6B.!CLR
- removed net N$9: IC5C.I0, IC5D.O
- new net 10H_A: 10H.1, 10HOURSA.CKB, 10HOURSA.QA, IC4A.I0, IC5A.I4, IC6A.!CLR, IC6A.!PRE, IC6A.J, IC6A.K, R9.2
- new net 12_HR: HOUR_SET.2, IC4A.O
- new net 24_HR: HOUR_SET.1, IC3B.O
- new net HR_RESET: 10HOURSA.R0(1), 10HOURSA.R0(2), HOURSA.R0(1), HOURSA.R0(2), HR_RESET.1
- net 10H_B: now also 10HOURSA.QB, IC3B.I1; no longer IC3B.I0, IC6B.!Q
- net 10M_C: now also HOUR_COUNT.1; no longer IC2B.I1
- net 10S_C: now also MIN_COUNT.1; no longer IC5A.I1
- net 1H_A: now also IC4A.I2, IC5A.I3; no longer IC4A.I1, IC7A.I1
- net 1H_B: now also IC4A.I1, IC5A.I2; no longer IC4A.I2, IC7A.I2
- net 1H_C: now also IC3B.I0, IC5A.I1; no longer IC3B.I1, IC7A.I3
- net 1H_D: now also 10HOURSA.CKA, IC5A.I0; no longer IC6B.CLK, IC7A.I4
- net AM: now also AM_PM.1; no longer JP1.1
- net GND: now also 10MINUTESA.R0(1), 10MINUTESA.R0(2), 10SECONDSA.R0(1), 10SECONDSA.R0(2), C1.-, MINUTESA.R0(1), MINUTESA.R0(2), POWER.2, SECONDSA.R0(1), SECONDSA.R0(2); no longer C1.2, C2.2, R5.1, R6.1, R7.1, R8.1, U$1G$1.!GAU
- net N$1: now also MIN_COUNT.2; no longer IC5A.O
- net N$15: now also CLOCK_IN.1; no longer IC2D.O
- net N$2: now also HOUR_SET.3, IC5A.O; no longer IC2C.O, IC5A.I0
- net N$21: now also HOUR_COUNT.2; no longer IC5B.O
- net PM: now also AM_PM.2; no longer JP1.2
- net VCC: now also C1.+, POWER.1; no longer R3.2, R4.2, SET.1, SET_HR.1, SET_MIN.1, U$1G$1.!CCLR, U$1G$1.!GAL, U$1G$1.!GBL, U$1G$1.!GBU
Other:
- note added: "INPUT=13"
- note added: "INPUT=24"
- note removed: "CLOCK PULSE"
- moved on the sheet: 10H, IC3B, IC4A, IC6A, R9

Commit message: clock pulse test new
Parts:
- removed AM_PM: (no value), iStivi - Header-Connector:M02PTH3
- removed HOUR_SET: (no value), iStivi - Header-Connector:M03LONGPADS
- removed IC3: 74LS08N, iStivi - ICs:74LS08N
- removed IC4: 74LS11N, iStivi - ICs:74LS11N
- removed IC5: 74S260D, iStivi - ICs:74S260D
- removed IC6: 74LS112D, iStivi - ICs:74LS112D
- removed R9: 10K, iStivi - RCLD:RESISTOR0207/7
- 10H: value (none) -> M02X2; device iStivi - Header-Connector:M02PTH3 -> iStivi - Header-Connector:M02X2
- 1H: value (none) -> M04X2; device iStivi - Header-Connector:M04LONGPADS -> iStivi - Header-Connector:M04X2
Connections:
- removed net 12_HR: HOUR_SET.2, IC4A.O
- removed net 24_HR: HOUR_SET.1, IC3B.O
- removed net AM: AM_PM.1, IC6A.Q
- removed net N$2: HOUR_SET.3, IC5A.O
- removed net PM: AM_PM.2, IC6A.!Q
- net 10H_A: now also 10H.2; no longer IC4A.I0, IC5A.I4, IC6A.!CLR, IC6A.!PRE, IC6A.J, IC6A.K, R9.2
- net 10H_B: now also 10H.3, 10H.4; no longer 10H.2, IC3B.I1
- net 1H_A: now also 1H.2; no longer IC4A.I2, IC5A.I3
- net 1H_B: now also 1H.3, 1H.4; no longer 1H.2, IC4A.I1, IC5A.I2
- net 1H_C: now also 1H.5, 1H.6; no longer 1H.3, IC3B.I0, IC5A.I1
- net 1H_D: now also 1H.7, 1H.8; no longer 1H.4, IC5A.I0
- net VCC: no longer R9.1
Other:
- note removed: "12 HOUR"
- note removed: "24 HOUR"
- note removed: "AM/PM"
- note removed: "INPUT=13"
- note removed: "INPUT=24"
