File: clock tests/clock_pulse_test.brd (EAGLE design)
At the start: 100 x 50 mm, 16 parts, among them IC1 74LS14N, Q1 32.768kHz

Commit message: clock pulse test new
Parts:
- IC1: value 74LS14N -> 74LS14D; device iStivi - ICs:DIL14 -> iStivi - ICs:SO14
- moved IN 37.5 mm to (38.7, 43.8)
- moved C1 24.8 mm to (15.9, 34.9), turned to 180 degrees
- moved C2 23.9 mm to (31.8, 34.9), turned to 90 degrees
- moved Q1 13.1 mm to (24.1, 29.8)
- moved OUT 10.2 mm to (64.8, 43.8)
- moved IC1 8.91 mm to (45.1, 17.8), turned to 0 degrees
- moved R2 8.64 mm to (29.8, 20.3), turned to 90 degrees
- moved U$2 7.18 mm to (87.0, 33.0)
- moved R1 6.98 mm to (17.8, 20.3), turned to 90 degrees
- moved R4 5.12 mm to (55.2, 34.9)
- moved R3 5.12 mm to (79.4, 39.4)
- moved U$1 1.42 mm to (69.2, 18.4)
Routing:
- net GND: track 163.3 -> 134.6 mm, vias 4 -> 1
- net N$14: track 71.9 -> 44.1 mm
- net VCC: track 106.5 -> 117.9 mm, vias 2 -> 0
- net N$16: track 34.2 -> 44.2 mm
- net N$8: track 7.62 -> 16.3 mm
- net N$5: track 7.62 -> 16.3 mm
- net N$1: track 7.62 -> 16.3 mm
- net N$7: track 7.62 -> 16.3 mm
- net N$6: track 7.62 -> 16.3 mm
- net N$4: track 7.62 -> 16.3 mm
- net N$3: track 7.62 -> 16.3 mm
- net N$2: track 7.62 -> 16.3 mm
- net N$11: track 37.8 -> 42.5 mm
- net N$13: track 27.8 -> 30.7 mm
- net N$12: track 13.3 -> 12.6 mm
Other:
- board text added: "CLOCK PULSE TEST"
