File: Double Tube/double-tube-base.brd (EAGLE design)
At the start: 52 x 42 mm, 9 parts

Commit message: Update some files
Parts:
- removed R2: 4k7, iStivi - RCLD:R0805
- added BC817: NPN_SMD, iStivi - Transistor-FET-reg:SOT-23
- added C1: 2n2, iStivi - RCLD:C0603K
- added C2: (no value), iStivi - RCLD:C1812K
- added C3: (no value), iStivi - RCLD:SMC_D
- added D1: (no value), iStivi - RCLD:SMA-DIODE
- added IC1: NE555D, iStivi - ICs:SO08
- added L1: (no value), iStivi - RCLD:SMD-10MM
- added R3: 1k, iStivi - RCLD:R0603
- added R4: 10k, iStivi - RCLD:R0603
- added R5: 56k, iStivi - RCLD:R0603
- added R6: 560k, iStivi - RCLD:R1206
- added R7: 5k, iStivi - RCLD:TRIM-EVM2N
- added U$5: FET-SOT223, iStivi - Transistor-FET-reg:SOT-223
- added U$6: (no value), iStivi - Logos:BUZZBOY
- added U$7: (no value), iStivi - Logos:BUZZBOY-SILK-BOTTOM
- JP3: value (none) -> M12PTH; device iStivi - Header-Connector:1X02 -> iStivi - Header-Connector:1X12
- R1: value 4k7 -> 1k1; device iStivi - RCLD:R0805 -> iStivi - RCLD:R1206
- moved JP3 42.0 mm to (53.3, 34.3), turned to 270 degrees
- moved R1 26.5 mm to (19.1, 7.62), turned to 180 degrees
Connections:
- removed net N1-DP: JP1.2, JP3.2, R2.1
- removed net N2-DP: JP1.1, JP3.1, R1.2
- new net N$1: IC1.7, R3.2, R4.1
- new net N$11: JP1.1, JP3.3
- new net N$12: JP1.3, JP3.4
- new net N$13: JP1.5, JP3.5
- new net N$14: JP1.7, JP3.6
- new net N$15: JP1.9, JP3.7
- new net N$16: JP1.2, JP3.8
- new net N$17: JP1.4, JP3.9
- new net N$18: JP1.6, JP3.10
- new net N$19: JP1.8, JP3.11
- new net N$2: C1.1, IC1.2, IC1.6, R4.2
- new net N$20: JP1.10, JP3.12
- new net N$3: BC817.1, IC1.5, R5.2
- new net N$4: D1.A, L1.P$2, U$5.2, U$5.4
- new net N$5: C2.1, D1.C, R1.2, R6.2
- new net N$6: BC817.3, R7.P$2
- new net N$7: R6.1, R7.P$1
- new net N$8: IC1.3, U$5.1
- new net N$9: JP2.3, R1.1
- new net VCC: C3.+, IC1.4, IC1.8, JP2.2, JP3.1, L1.P$1, R3.1, R5.1
- net GND: now also BC817.2, C1.2, C2.2, C3.-, IC1.1, JP2.1, JP3.2, R7.P$3, U$5.3; no longer R1.1, R2.2
Routing:
- net GND: track 0.00 -> 108.0 mm, vias 0 -> 6
- net N$17: track 0.00 -> 103.9 mm
- net N$16: track 0.00 -> 96.0 mm
- net VCC: track 0.00 -> 95.4 mm, vias 0 -> 3
- net N$11: track 0.00 -> 92.4 mm, vias 0 -> 4
- net N$12: track 0.00 -> 64.9 mm, vias 0 -> 4
- net N$13: track 0.00 -> 64.7 mm, vias 0 -> 3
- net N$18: track 0.00 -> 58.6 mm, vias 0 -> 1
- net N$20: track 0.00 -> 57.9 mm
- net N$19: track 0.00 -> 56.8 mm, vias 0 -> 1
- net N$1: track 0.00 -> 33.9 mm, vias 0 -> 2
- net N$8: track 0.00 -> 32.1 mm, vias 0 -> 2
- net N$14: track 0.00 -> 30.7 mm, vias 0 -> 1
- net N$3: track 0.00 -> 29.4 mm, vias 0 -> 2
- net N$15: track 0.00 -> 29.2 mm
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Other:
- board size 52 x 42 mm -> 58.4 x 42 mm
- board text added: "+"
- board text added: "A"
- board text added: "B"
- board text added: "C"
- board text added: "D"
- board text added: "DUAL TUBE POWER PROTOTYPE"
- board text added: "G"
- board text added: "P"
- board text added: "V"
