File: Double Tube/double-tube.brd (EAGLE design)
At the start: 52 x 42 mm, 66 parts, among them IC1 4028D, IC2 4028D

Commit message: double
Connections:
- net GND: now also R27.1, R28.1
- net VCC: no longer R27.1, R28.1
Routing:
- net VCC: track 67.4 -> 61.4 mm
- net GND: track 193.9 -> 197.8 mm
Changed lines of the file:
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@@
 <via x="29.972" y="16.6624" extent="1-16" drill="0.4"/>
 <via x="29.464" y="18.8976" extent="1-16" drill="0.4"/>
+<contactref element="R27" pad="1"/>
+<contactref element="R28" pad="1"/>
+<wire x1="27.0256" y1="29.2608" x2="27.09" y2="29.21" width="0.254" layer="1"/>
+<wire x1="24.98" y1="29.21" x2="25.2984" y2="29.21" width="0.254" layer="1"/>
+<wire x1="25.2984" y1="29.21" x2="25.2984" y2="27.8384" width="0.254" layer="1"/>
+<wire x1="24.98" y1="29.21" x2="27.09" y2="29.21" width="0.254" layer="1"/>
 </signal>
 <signal name="N$1">
@@
 <contactref element="R25" pad="1"/>
 <contactref element="R26" pad="1"/>
-<contactref element="R27" pad="1"/>
-<contactref element="R28" pad="1"/>
 <contactref element="R29" pad="1"/>
 <contactref element="R30" pad="1"/>
@@
 <wire x1="27.1272" y1="21.5392" x2="27.09" y2="21.59" width="0.254" layer="1"/>
 <wire x1="27.1272" y1="17.8816" x2="27.09" y2="17.78" width="0.254" layer="1"/>
-<wire x1="27.1272" y1="29.1592" x2="27.1272" y2="25.4" width="0.254" layer="1"/>
 <wire x1="27.1272" y1="25.4" x2="27.09" y2="25.4" width="0.254" layer="1"/>
-<wire x1="27.1272" y1="29.1592" x2="27.09" y2="29.21" width="0.254" layer="1"/>
-<wire x1="27.0256" y1="29.2608" x2="24.9936" y2="29.2608" width="0.254" layer="1"/>
-<wire x1="24.9936" y1="29.2608" x2="24.98" y2="29.21" width="0.254" layer="1"/>
-<wire x1="27.0256" y1="29.2608" x2="27.09" y2="29.21" width="0.254" layer="1"/>
 <wire x1="24.9936" y1="17.78" x2="24.9936" y2="14.0208" width="0.254" layer="1"/>
 <wire x1="24.9936" y1="14.0208" x2="24.98" y2="13.97" width="0.254" layer="1"/>
