File: 180V_power/180V_power.sch (EAGLE design)
At the start: 18 parts, among them IC1 NE555P, Q1 IRF740S, Q2 BC546

Commit message: new 180v board
Parts:
- L1: device iStivi - RCLD:INDUCTOR0207/10 -> iStivi - RCLD:INDUCTORTFI0307
Changed lines of the file:
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@@
 <part name="Q2" library="iStivi - Transistor-FET" deviceset="BC546*" device="" technology="B" value="BC546"/>
 <part name="C2" library="iStivi - RCLD" deviceset="CAPACITOR" device="C1206K" value="2n2"/>
-<part name="L1" library="iStivi - RCLD" deviceset="INDUCTOR" device="0207/10" value="100uH"/>
+<part name="L1" library="iStivi - RCLD" deviceset="INDUCTOR" device="TFI0307" value="100uH"/>
 <part name="VR1" library="iStivi - RCLD" deviceset="TRIM_POT" device="CA6V" value="1K"/>
 <part name="GND1" library="iStivi - Supply" deviceset="GND" device=""/>

Commit message: new 180V and tube tester
Parts:
- Q2: device iStivi - Transistor-FET:BC546B -> iStivi - Transistor-FET-reg:BC546A
Changed lines of the file:
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@@
 <part name="R6" library="iStivi - RCLD" deviceset="RESISTOR" device="R1206" value="2K2"/>
 <part name="C3" library="iStivi - RCLD" deviceset="CAPACITOR" device="C1206K" value="100pF"/>
-<part name="Q2" library="iStivi - Transistor-FET" deviceset="BC546*" device="" technology="B" value="BC546"/>
+<part name="Q2" library="iStivi - Transistor-FET-reg" deviceset="BC546*" device="" technology="A" value="BC546"/>
 <part name="C2" library="iStivi - RCLD" deviceset="CAPACITOR" device="C1206K" value="2n2"/>
 <part name="L1" library="iStivi - RCLD" deviceset="INDUCTOR" device="TFI0307" value="100uH"/>

Commit message: new simple 180 board
Parts:
- removed IN: POWER_JACKSLT, iStivi - Header-Connector:POWER_JACKSLT
- added JP1: (no value), iStivi - Header-Connector:M023.5MM
- C2, C3: device iStivi - RCLD:CAPACITORC1206K -> iStivi - RCLD:CAPACITOR050-025X075
- D1: device iStivi - RCLD:DIODESMA -> iStivi - RCLD:DIODEPTH
- L1: value 100uH -> (none); device iStivi - RCLD:INDUCTORTFI0307 -> iStivi - RCLD:INDUCTOR
- Q1: value IRF740S -> IRF740; device iStivi - Transistor-FET:IRF740S -> iStivi - Transistor-FET:IRF740
- R1, R2, R3, R6: device iStivi - RCLD:RESISTORR1206 -> iStivi - RCLD:RESISTOR0207/10
Connections:
- net GND: now also JP1.2; no longer IN.GND, IN.GNDBREAK
- net N$26: now also JP1.1; no longer IN.PWR
